File: PCB/miernik/miernik.kicad_pcb (KiCad board)
At the start: 2 copper layers, 40 parts, among them J1 Conn_01x01, J10 Conn_01x01, J11 Conn_01x01, J12 Conn_01x01, J2 Conn_01x01, J3 Conn_01x01, J4 Conn_01x01, J5 Conn_01x01, J6 Conn_01x01, J7 Conn_01x01, J8 Conn_01x01, J9 Conn_01x01, Q1 MMBTA42, Q2 MMBTA42, Q3 MMBTA42, SW1 SW_Push, SW2 SW_Push, SW3 SW_Push, U1 ATmega8-16PU, U2 3DIGIT-7SEGMENT, U3 A1101ELHL, Y1 Crystal

Commit message: Add files via upload
Added temperature sensor, added some letters and names for modes, fixed problem with float in total distance.
Parts:
- added U2: TMP36, Package_TO_SOT_THT:TO-92, F.Cu at (134.9, 150.1)
- renumbered J11 to J1, J9 to J10, J10 to J11, J1 to J2, J2 to J3, J3 to J4, J4 to J5, J5 to J6, J6 to J7, J7 to J8, J8 to J9, R12 to R10, R13 to R11, R3 to R12, R4 to R13, R5 to R14, R14 to R2, R2 to R3, R6 to R4, R7 to R5, R8 to R6, R9 to R7, R10 to R8, R11 to R9, U2 to U4
Connections:
- U1 pad 27: (no net) -> Net-(U1-Pad27)
Routing:
- net +5V: track 53.6 -> 90.6 mm
- net Net-(U1-Pad27): track 0.00 -> 30.4 mm
- net GND: track 128.0 -> 131.2 mm
- net Net-(J5-Pad1): track 15.0 -> 16.3 mm
- net Net-(C1-Pad2): track 31.4 -> 32.3 mm
- net Net-(SW3-Pad1): track 17.2 -> 16.3 mm
Other:
- net class Default: via_dia 0.8 -> 1.2
- net class Pwr added: clearance 0.5, trace_width 1, via_dia 1.2, via_drill 0.4
- net class Signal added: clearance 0.3, trace_width 0.7, via_dia 1, via_drill 0.4
- net class nowe removed
- board text added: "Kolikon 2020"
